File: hw/Control_PCB/Control_PCB.kicad_pcb (KiCad board)
At the start: 2 copper layers, 37 x 15.3 mm, 15 parts, among them J1 USB_C_Receptacle_PowerOnly_6P, J2 Conn_01x04, J3 Conn_01x03_Pin, SW1 Brightness, SW2 Mode, U1 ATtiny816-M

Commit message: PCB release to manufacturing
Parts:
- added R5: 1k, Resistor_SMD:R_0603_1608Metric, F.Cu at (137.1, 68.3)
- added TP1: Tick, TestPoint:TestPoint_Pad_D1.0mm, B.Cu at (143.3, 61.0)
- moved U1 0.11 mm to (142.3, 63.5)
Connections:
- J2 pad 1: /DATA -> GND
- J2 pad 2: VBUS -> /CLK
- J2 pad 3: GND -> /DATA
- J2 pad 4: /CLK -> VBUS
- U1 pad 1: unconnected-(U1-PA2-Pad1) -> /mode
- U1 pad 10: unconnected-(U1-PB4-Pad10) -> /DATA
- U1 pad 14: unconnected-(U1-PB0-Pad14) -> /brightness
- U1 pad 15: unconnected-(U1-PC0-Pad15) -> Net-(U1-PC0)
- U1 pad 19: unconnected-(U1-~{RESET}/PA0-Pad19) -> Net-(U1-~{RESET}/PA0)
- U1 pad 9: unconnected-(U1-PB5-Pad9) -> /CLK
Routing:
- net /brightness: track 0.00 -> 25.2 mm
- net VBUS: track 26.0 -> 44.5 mm, vias 0 -> 2
- net /UPDI: track 0.00 -> 14.6 mm
- net /DATA: track 0.00 -> 12.7 mm, vias 0 -> 2
- net /CLK: track 0.00 -> 12.6 mm, vias 0 -> 2
- net /mode: track 0.00 -> 11.5 mm
- net Net-(U1-~{RESET}/PA0): track 0.00 -> 10.7 mm, vias 0 -> 2
- net GND: track 0.00 -> 2.48 mm, vias 1 -> 18
- net Net-(U1-PC0): track 0.00 -> 1.91 mm, vias 0 -> 1
Other:
- board text added: "GND UPDI +5V"
- board text added: "Tick"
- board text removed: "GND UDPI +5V"

Commit message: BOM complete
Parts:
- J1: value USB_C_Receptacle_PowerOnly_6P -> USB4125-GF-A
- J2: value Conn_01x04 -> PRPC040DAAN-RC
- U1: value ATtiny816-M -> ATtiny1616-M
