File: hw/Control_PCB/Control_PCB.kicad_sch (KiCad schematic)
At the start: 13 parts, among them J1 USB_C_Receptacle_PowerOnly_6P, J2 Conn_01x04, J3 Conn_01x03_Pin, SW1 Brightness, SW2 Mode, U1 ATtiny816-M

Commit message: PCB release to manufacturing
Parts:
- added R5: 1k, Resistor_SMD:R_0603_1608Metric, symbol Device:R_Small_US
- added TP1: Tick, TestPoint:TestPoint_Pad_D1.0mm, symbol Connector:TestPoint
- J1: value USB_C_Receptacle_PowerOnly_6P -> USB4125-GF-A
Connections:
- net CLK: now also J2.2 (Pin_2), U1.9 (PB5); no longer J2.4 (Pin_4)
- net DATA: now also J2.3 (Pin_3), U1.10 (PB4); no longer J2.1 (Pin_1)
- net GND: now also J2.1 (Pin_1); no longer J2.3 (Pin_3)
- net UPDI: now also R5.2
- net VBUS: now also J2.4 (Pin_4); no longer J2.2 (Pin_2)
- net brightness: now also U1.14 (PB0)
- net mode: now also U1.1 (PA2)
- net at U1.15 (PC0): now also TP1.1
- net at U1.19 (~{RESET}/PA0): now also R5.1
Other:
- moved on the sheet: C2, U1

Commit message: BOM complete
Parts:
- removed U1: ATtiny816-M, Package_DFN_QFN:VQFN-20-1EP_3x3mm_P0.4mm_EP1.7x1.7mm, symbol MCU_Microchip_ATtiny:ATtiny816-M
- added U1: ATtiny1616-M, Package_DFN_QFN:VQFN-20-1EP_3x3mm_P0.4mm_EP1.7x1.7mm, symbol MCU_Microchip_ATtiny:ATtiny1616-M
- J2: value Conn_01x04 -> PRPC040DAAN-RC
Connections:
- net CLK: now also U1.9 (PB5)
- net DATA: now also U1.10 (PB4)
- net GND: now also U1.21 (GND), U1.3 (GND)
- net VBUS: now also U1.4 (VCC)
- net brightness: now also U1.14 (PB0)
- net mode: now also U1.1 (PA2)
- net at R5.1: now also U1.19 (~{RESET}/PA0)
- net at TP1.1: now also U1.15 (PC0)
Changed lines of the file:
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@@
 			)
 		)
-		(property "Value" "Conn_01x04"
+		(property "Value" "PRPC040DAAN-RC"
 			(at 123.19 49.5301 0)
 			(effects
@@
 				(path "/def01542-b5e0-4a62-8767-06e1293c8ead"
 					(reference "J1")
+					(unit 1)
+				)
+			)
+		)
+	)
+	(symbol
+		(lib_id "MCU_Microchip_ATtiny:ATtiny1616-M")
+		(at 185.42 109.22 0)
+		(unit 1)
+		(exclude_from_sim no)
+		(in_bom yes)
+		(on_board yes)
+		(dnp no)
+		(fields_autoplaced yes)
+		(property "Reference" "U1"
+			(at 187.5633 83.82 0)
+			(effects
+				(font
+					(size 1.27 1.27)
+				)
+				(justify left)
+			)
+		)
+		(property "Value" "ATtiny1616-M"
+			(at 187.5633 86.36 0)
+			(effects
+				(font
+					(size 1.27 1.27)
+				)
+				(justify left)
+			)
+		)
+		(property "Footprint" "Package_DFN_QFN:VQFN-20-1EP_3x3mm_P0.4mm_EP1.7x1.7mm"
+			(at 185.42 109.22 0)
+			(effects
+				(font
+					(size 1.27 1.27)
+					(italic yes)
+				)
+				(hide yes)
+			)
+		)
+		(property "Datasheet" "http://ww1.microchip.com/downloads/en/DeviceDoc/ATtiny3216_ATtiny1616-data-sheet-40001997B.pdf"
+			(at 185.42 109.22 0)
+			(effects
+				(font
+					(size 1.27 1.27)
+				)
+				(hide yes)
+			)
+		)
+		(property "Description" "20MHz, 16kB Flash, 2kB SRAM, 256B EEPROM, VQFN-20"
+			(at 185.42 109.22 0)
+			(effects
+				(font
+					(size 1.27 1.27)
+				)
+				(hide yes)
+			)
+		)
+		(pin "3"
+		)
+		(pin "15"
+		)
+		(pin "16"
+		)
+		(pin "17"
+		)
+		(pin "18"
+		)
+		(pin "10"
+		)
+		(pin "4"
+		)
+		(pin "21"
+		)
+		(pin "20"
+		)
+		(pin "7"
+		)
+		(pin "8"
+		)
+		(pin "2"
+		)
+		(pin "14"
+		)
+		(pin "5"
+		)
+		(pin "13"
+		)
+		(pin "19"
+		)
+		(pin "12"
+		)
+		(pin "11"
+		)
+		(pin "1"
+		)
+		(pin "9"
+		)
+		(pin "6"
+		)
+		(instances
+			(project ""
+				(path "/def01542-b5e0-4a62-8767-06e1293c8ead"
+					(reference "U1")
 					(unit 1)
 				)
@@
 					(unit 1)
 				)
-			)
-		)
-	)
-	(symbol
-		(lib_id "MCU_Microchip_ATtiny:ATtiny816-M")
-		(at 185.42 109.22 0)
-		(unit 1)
-		(exclude_from_sim no)
-		(in_bom yes)
-		(on_board yes)
-		(dnp no)
-		(fields_autoplaced yes)
-		(property "Reference" "U1"
-			(at 187.5633 83.82 0)
-			(effects
-				(font
-					(size 1.27 1.27)
-				)
-				(justify left)
-			)
-		)
-		(property "Value" "ATtiny816-M"
-			(at 187.5633 86.36 0)
-			(effects
-				(font
-					(size 1.27 1.27)
-				)
-				(justify left)
-			)
-		)
-		(property "Footprint" "Package_DFN_QFN:VQFN-20-1EP_3x3mm_P0.4mm_EP1.7x1.7mm"
-			(at 185.42 109.22 0)
-			(effects
-				(font
-					(size 1.27 1.27)
-					(italic yes)
-				)
-				(hide yes)
-			)
-		)
-		(property "Datasheet" "http://ww1.microchip.com/downloads/en/DeviceDoc/40001913A.pdf"
-			(at 185.42 109.22 0)
-			(effects
-				(font
-					(size 1.27 1.27)
-				)
-				(hide yes)
-			)
-		)
-		(property "Description" "20MHz, 8kB Flash, 512B SRAM, 128B EEPROM, VQFN-20"
-			(at 185.42 109.22 0)
-			(effects
-				(font
-					(size 1.27 1.27)
-				)
-				(hide yes)
-			)
-		)
-		(pin "17"
-		)
-		(pin "12"
-		)
-		(pin "19"
-		)
-		(pin "16"
-		)
-		(pin "15"
-		)
-		(pin "5"
-		)
-		(pin "3"
-		)
-		(pin "6"
-		)
-		(pin "18"
-		)
-		(pin "20"
-		)
-		(pin "8"
-		)
-		(pin "21"
-		)
-		(pin "2"
-		)
-		(pin "14"
-		)
-		(pin "4"
-		)
-		(pin "1"
-		)
-		(pin "13"
-		)
-		(pin "7"
-		)
-		(pin "11"
-		)
-		(pin "10"
-		)
-		(pin "9"
-		)
-		(instances
-			(project ""
-				(path "/def01542-b5e0-4a62-8767-06e1293c8ead"
-					(reference "U1")
-					(unit 1)
-				)

Commit message: Change UPDI buffer resistor to 0 Ohms. Internet recommendation of 1k didn't work. Not sure this is needed because of diode on UPDI 5V rail.
Parts:
- R5: value 1k -> 0
Changed lines of the file:
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@@
 			)
 		)
-		(property "Value" "1k"
+		(property "Value" "0"
 			(at 207.01 90.424 0)
 			(effects
