File: hw/LED_PCB/LED_PCB.kicad_pcb (KiCad board)
At the start: 2 copper layers, 64 x 64 mm, 17 parts, among them J1 Conn_01x04

Commit message: PCB release to manufacturing
Routing:
- net Net-(D1-CI): track 5.87 -> 5.23 mm
Changed lines of the file:
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@@
 		(pcbplotparams
 			(layerselection 0x00000000_00000000_55555555_5755f5ff)
-			(plot_on_all_layers_selection 0x00000000_00000000_00000000_00000000)
+			(plot_on_all_layers_selection 0x00000000_00000000_00000000_02000000)
 			(disableapertmacros no)
 			(usegerberextensions no)
@@
 			(outputformat 1)
 			(mirror no)
-			(drillshape 1)
+			(drillshape 0)
 			(scaleselection 1)
-			(outputdirectory "")
+			(outputdirectory "manufacturing/")
 		)
 	)
@@
 		(net 4)
 	)
-	(segment
-		(start 146.0644 71.7032)
-		(end 146.514448 72.153248)
-		(width 0.2032)
-		(layer "B.Cu")
-		(net 4)
-	)

Commit message: BOM complete
Parts:
- J1: value Conn_01x04 -> PPPC022LFBN-RC
Changed lines of the file:
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@@
 			)
 		)
-		(property "Value" "Conn_01x04"
+		(property "Value" "PPPC022LFBN-RC"
 			(at -1.27 -5.31 90)
 			(layer "B.Fab")
