File: hw/LED_PCB/LED_PCB.kicad_sch (KiCad schematic)
At the start: 15 parts, among them J1 Conn_01x04

Commit message: BOM complete
Parts:
- J1: value Conn_01x04 -> PPPC022LFBN-RC
Changed lines of the file:
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@@
 			)
 		)
-		(property "Value" "Conn_01x04"
+		(property "Value" "PPPC022LFBN-RC"
 			(at 21.59 74.93 0)
 			(effects
